File: interface-full.kicad_pcb (KiCad board)
At the start: 2 copper layers, 218.6 x 65 mm, 57 parts, among them J1 RASPBERRY PI, J10 RPI_RX, J11 GND, J12 GND, J13 RX, J14 TX, J15 GND, J16 RX, J17 TX, J18 GND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

Commit message: board done
Parts:
- added REF**: MountingHole_3.2mm_M3_ISO14580_Pad, MountingHole:MountingHole_3.2mm_M3_ISO14580_Pad, F.Cu at (83.2, 79.4)
- Raspberry PI: renamed from REF**
Routing:
- net RPI_5V: track 202.6 -> 205.9 mm
Other:
- board text added: "Home Assistant Lighting Interface Daniel Mazzer - 02/2020"
- board text removed: "Layout based on mechanical drawings at: https://www.raspberrypi.org/documentation/hardware/raspberrypi/mechanical/README.md"
