File: board/interface-full.kicad_pcb (KiCad board)
At the start: 2 copper layers, 218.6 x 65 mm, 58 parts, among them J1 RASPBERRY PI, J10 RPI_RX, J11 GND, J12 GND, J13 RX, J14 TX, J15 GND, J16 RX, J17 TX, J18 GND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

Commit message: change sch to match rpi gpio numbering
Connections:
- net RPI_GPIO_0 renamed RPI_GPIO_17
- net RPI_GPIO_1 renamed RPI_GPIO_18
- net RPI_GPIO_28 renamed RPI_GPIO_20
- A1 pad 10: RPI_GPIO_3 -> RPI_GPIO_22
- A1 pad 11: RPI_GPIO_12 -> RPI_GPIO_10
- A1 pad 12: RPI_GPIO_13 -> RPI_GPIO_09
- A1 pad 9: RPI_GPIO_2 -> RPI_GPIO_27
- A2 pad 10: RPI_GPIO_25 -> RPI_GPIO_26
- A2 pad 12: RPI_GPIO_4 -> RPI_GPIO_23
- A2 pad 9: RPI_GPIO_24 -> RPI_GPIO_19
- A3 pad 10: RPI_GPIO_27 -> RPI_GPIO_16
- A3 pad 12: RPI_GPIO_29 -> RPI_GPIO_21
- A3 pad 9: RPI_GPIO_26 -> RPI_GPIO_12
- J1 pad 10: RPI_GPIO_16 -> RPI_GPIO_15
- J1 pad 13: RPI_GPIO_2 -> RPI_GPIO_27
- J1 pad 15: RPI_GPIO_3 -> RPI_GPIO_22
- J1 pad 16: RPI_GPIO_4 -> RPI_GPIO_23
- J1 pad 18: RPI_GPIO_5 -> RPI_GPIO_24
- J1 pad 19: RPI_GPIO_12 -> RPI_GPIO_10
- J1 pad 21: RPI_GPIO_13 -> RPI_GPIO_09
- J1 pad 22: RPI_GPIO_6 -> RPI_GPIO_25
- J1 pad 23: RPI_GPIO_14 -> RPI_GPIO_11
- J1 pad 24: RPI_GPIO_10 -> RPI_GPIO_8
- J1 pad 26: RPI_GPIO_11 -> RPI_GPIO_7
- J1 pad 29: RPI_GPIO_21 -> RPI_GPIO_5
- J1 pad 3: RPI_GPIO_8 -> RPI_GPIO_2
- J1 pad 31: RPI_GPIO_22 -> RPI_GPIO_6
- J1 pad 32: RPI_GPIO_26 -> RPI_GPIO_12
- J1 pad 33: RPI_GPIO_23 -> RPI_GPIO_13
- J1 pad 35: RPI_GPIO_24 -> RPI_GPIO_19
- J1 pad 36: RPI_GPIO_27 -> RPI_GPIO_16
- J1 pad 37: RPI_GPIO_25 -> RPI_GPIO_26
- J1 pad 40: RPI_GPIO_29 -> RPI_GPIO_21
- J1 pad 5: RPI_GPIO_9 -> RPI_GPIO_3
- J1 pad 7: RPI_GPIO_7 -> RPI_GPIO_4
- J1 pad 8: RPI_GPIO_15 -> RPI_GPIO_14
- J10 pad 1: RPI_GPIO_16 -> RPI_GPIO_15
- J8 pad 1: RPI_GPIO_15 -> RPI_GPIO_14
- R11 pad 2: RPI_GPIO_14 -> RPI_GPIO_11
- R12 pad 2: RPI_GPIO_21 -> RPI_GPIO_5
- R13 pad 2: RPI_GPIO_22 -> RPI_GPIO_6
- R14 pad 2: RPI_GPIO_23 -> RPI_GPIO_13
- R15 pad 1: RPI_GPIO_14 -> RPI_GPIO_11
- R16 pad 1: RPI_GPIO_21 -> RPI_GPIO_5
- R17 pad 1: RPI_GPIO_22 -> RPI_GPIO_6
- R18 pad 1: RPI_GPIO_23 -> RPI_GPIO_13
- R2 pad 2: RPI_GPIO_8 -> RPI_GPIO_2
- R20 pad 2: RPI_GPIO_5 -> RPI_GPIO_24
- R21 pad 2: RPI_GPIO_6 -> RPI_GPIO_25
- R22 pad 2: RPI_GPIO_10 -> RPI_GPIO_8
- R23 pad 2: RPI_GPIO_11 -> RPI_GPIO_7
- R24 pad 1: RPI_GPIO_5 -> RPI_GPIO_24
- R25 pad 1: RPI_GPIO_6 -> RPI_GPIO_25
- R26 pad 1: RPI_GPIO_10 -> RPI_GPIO_8
- R27 pad 1: RPI_GPIO_11 -> RPI_GPIO_7
- R3 pad 2: RPI_GPIO_9 -> RPI_GPIO_3
- R4 pad 2: RPI_GPIO_7 -> RPI_GPIO_4
- R6 pad 1: RPI_GPIO_8 -> RPI_GPIO_2
- R7 pad 1: RPI_GPIO_9 -> RPI_GPIO_3
- R8 pad 1: RPI_GPIO_7 -> RPI_GPIO_4
Routing:
- net RPI_GPIO_09: track 0.00 -> 167.5 mm, vias 0 -> 2
- net RPI_GPIO_9: track 158.1 -> 0.00 mm, vias 2 -> 0
- net RPI_GPIO_13: track 167.5 -> 34.6 mm, vias 2 -> 0
- net RPI_GPIO_22: track 40.1 -> 159.7 mm, vias 2 -> 0
- net RPI_GPIO_29: track 111.3 -> 0.00 mm, vias 2 -> 0
- net RPI_GPIO_19: track 0.00 -> 97.2 mm, vias 0 -> 1
- net RPI_GPIO_16: track 16.8 -> 110.4 mm, vias 0 -> 2
- net RPI_GPIO_5: track 112.3 -> 45.3 mm
- net RPI_GPIO_6: track 106.7 -> 40.1 mm
- net RPI_GPIO_21: track 45.3 -> 111.3 mm
- net RPI_GPIO_7: track 151.9 -> 86.6 mm, vias 4 -> 2
- net RPI_GPIO_23: track 34.6 -> 98.4 mm, vias 0 -> 3
- net RPI_GPIO_10: track 103.2 -> 166.0 mm
- net RPI_GPIO_8: track 165.1 -> 103.2 mm, vias 4 -> 2
- net RPI_GPIO_12: track 166.0 -> 107.8 mm
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